Commit message: Update AA-pro.urdf

File: AA-pro.urdf (robot description, URDF)
Before this commit: robot robot_arm, 8 links, 5 joints
Joints:
- joint base_joint: axis 0 0 1 -> 0 0 -1
- joint elbow_joint: limit lower=-1.57 upper=1.57 -> lower=-1.14 upper=2
- joint elbow_joint22: axis -1 0 0 -> 1 0 0
- joint shoulder_joint: limit lower=-1.57 upper=1.57 -> lower=-1.14 upper=2
